Commit message: add RL version urdf

File: urdf/h1.urdf (robot description, URDF)
Before this commit: robot H1, 25 links, 24 joints
Links:
- removed link d435_left_imager_link
- removed link d435_rgb_module_link
- removed link logo_link
- removed link mid360_link
- link left_ankle_link: geometry collision box size=0.29 0.03 0.024; visual mesh filename=package://h1_description/meshes/left_ankle_link.dae
- link left_hip_pitch_link: mass 4.152 -> 6.1
- link left_knee_link: mass 1.721 -> 2.3
- link pelvis: mass 5.39 -> 8.3
- link right_ankle_link: geometry collision box size=0.29 0.03 0.024; visual mesh filename=package://h1_description/meshes/right_ankle_link.dae
- link right_hip_pitch_link: mass 4.152 -> 6.1
- link right_knee_link: mass 1.721 -> 2.3
- link torso_link: mass 17.789 -> 20.8
Joints:
- removed joint d435_left_imager_joint
- removed joint d435_rgb_module_joint
- removed joint logo_joint
- removed joint mid360_joint

Commit message: add hands

File: urdf/h1.urdf (robot description, URDF)
Before this commit: robot H1, 21 links, 20 joints
Links:
- added link left_hand_link
- added link right_hand_link
Joints:
- added joint left_hand_joint: type fixed, parent left_elbow_link, child left_hand_link, origin xyz=0.2605 0 -0.0185 rpy=0 0 0, axis 1 0 0
- added joint right_hand_joint: type fixed, parent right_elbow_link, child right_hand_link, origin xyz=0.2605 0 -0.0185 rpy=0 0 0, axis 1 0 0

Commit message: Add ball hands + better convex

File: urdf/h1.urdf (robot description, URDF)
Before this commit: robot H1, 23 links, 22 joints
Links:
- link left_ankle_link: geometry visual mesh filename=package://h1_description/meshes/left_ankle_link.dae
- link left_elbow_link: geometry visual mesh filename=package://h1_description/meshes/left_elbow_link.dae
- link left_hip_pitch_link: geometry visual mesh filename=package://h1_description/meshes/left_hip_pitch_link.dae
- link left_hip_roll_link: geometry visual mesh filename=package://h1_description/meshes/left_hip_roll_link.dae
- link left_hip_yaw_link: geometry visual mesh filename=package://h1_description/meshes/left_hip_yaw_link.dae
- link left_knee_link: geometry visual mesh filename=package://h1_description/meshes/left_knee_link.dae
- link left_shoulder_pitch_link: geometry visual mesh filename=package://h1_description/meshes/left_shoulder_pitch_link.dae
- link left_shoulder_roll_link: geometry visual mesh filename=package://h1_description/meshes/left_shoulder_roll_link.dae
- link left_shoulder_yaw_link: geometry visual mesh filename=package://h1_description/meshes/left_shoulder_yaw_link.dae
- link pelvis: geometry visual mesh filename=package://h1_description/meshes/pelvis.dae
- link right_ankle_link: geometry visual mesh filename=package://h1_description/meshes/right_ankle_link.dae
- link right_elbow_link: geometry visual mesh filename=package://h1_description/meshes/right_elbow_link.dae
- link right_hip_pitch_link: geometry visual mesh filename=package://h1_description/meshes/right_hip_pitch_link.dae
- link right_hip_roll_link: geometry visual mesh filename=package://h1_description/meshes/right_hip_roll_link.dae
- link right_hip_yaw_link: geometry visual mesh filename=package://h1_description/meshes/right_hip_yaw_link.dae
- link right_knee_link: geometry visual mesh filename=package://h1_description/meshes/right_knee_link.dae
- link right_shoulder_pitch_link: geometry visual mesh filename=package://h1_description/meshes/right_shoulder_pitch_link.d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
- link right_shoulder_roll_link: geometry visual mesh filename=package://h1_description/meshes/right_shoulder_roll_link.dae
- link right_shoulder_yaw_link: geometry visual mesh filename=package://h1_description/meshes/right_shoulder_yaw_link.dae
- link torso_link: geometry visual mesh filename=package://h1_description/meshes/torso_link.dae
